Commit message: urdf done

File: install/amphibious_robot_description/share/amphibious_robot_description/description/amphibot.urdf.xacro (robot description, xacro)
@@ -4,6 +4,6 @@
        <color rgba="1 1 1 1" />
    </material>
-   <material name="black">
-       <color rgba="0 0 0 1" />
+   <material name="red">
+       <color rgba="1.0 0.0 0.0 1.0" />
    </material>
    <material name="blue">
@@ -26,8 +26,13 @@
      </geometry>
      <material name="white"/>
+     <gazebo>
+      <material>Gazebo/White</material>
+      <kp>1000000.0</kp>
+      <kd>100.0</kd>
+    </gazebo>
    </collision>
    <inertial>
-     <mass value="1.5"/>
-     <inertia ixx="0.02" ixy="0.0" ixz="0.0" iyy="0.02" iyz="0.0" izz="0.02"/>
+    <mass value="4.8"/>
+      <inertia ixx="0.0612" ixy="0.0" ixz="0.0" iyy="0.06948" iyz="0.0" izz="0.0954"/>
    </inertial>
  </link>
@@ -45,8 +50,13 @@
      </geometry>
      <material name="blue"/>
+     <gazebo>
+      <material>Gazebo/Blue</material>
+      <kp>1000000.0</kp>
+      <kd>100.0</kd>
+    </gazebo>
    </collision>
    <inertial>
-     <mass value="0.2"/>
-     <inertia ixx="0.001" ixy="0.0" ixz="0.0" iyy="0.001" iyz="0.0" izz="0.001"/>
+     <mass value="0.1"/>
+     <inertia ixx="0.00133" ixy="0.0" ixz="0.0" iyy="0.00133" iyz="0.0" izz="0.0000003125"/>
    </inertial>
  </link>
@@ -69,8 +79,13 @@
      </geometry>
      <material name="blue"/>
+     <gazebo>
+      <material>Gazebo/Blue</material>
+      <kp>1000000.0</kp>
+      <kd>100.0</kd>
+    </gazebo>
    </collision>
    <inertial>
-     <mass value="0.2"/>
-     <inertia ixx="0.001" ixy="0.0" ixz="0.0" iyy="0.001" iyz="0.0" izz="0.001"/>
+     <mass value="0.1"/>
+     <inertia ixx="0.00133" ixy="0.0" ixz="0.0" iyy="0.00133" iyz="0.0" izz="0.0000003125"/>
    </inertial>
  </link>
@@ -86,5 +101,5 @@
        <mesh filename="${mesh_path}/left_wheel.stl" scale="${scale_mm_to_m} ${scale_mm_to_m} ${scale_mm_to_m}"/>
      </geometry>
-     <material name="black"/>
+     <material name="red"/>
    </visual>
    <collision>
@@ -92,9 +107,21 @@
        <mesh filename="${mesh_path}/left_wheel.stl" scale="${scale_mm_to_m} ${scale_mm_to_m} ${scale_mm_to_m}"/>
      </geometry>
-     <material name="black"/>
+     <material name="red"/>
+     <gazebo>
+      <material>Gazebo/Red</material>
+      <friction>
+        <ode>
+          <mu>1.0</mu>
+          <mu2>1.0</mu2>
+          <fdir1>0 1 0</fdir1>
+        </ode>
+      </friction>
+      <kp>1000000.0</kp>
+      <kd>100.0</kd>
+    </gazebo>
    </collision>
    <inertial>
-     <mass value="0.3"/>
-     <inertia ixx="0.001" ixy="0.0" ixz="0.0" iyy="0.001" iyz="0.0" izz="0.001"/>
+     <mass value="0.5"/>
+     <inertia ixx="0.00733" ixy="0.0" ixz="0.0" iyy="0.00733" iyz="0.0" izz="0.00133"/>
    </inertial>
  </link>
@@ -111,5 +138,5 @@
        <mesh filename="${mesh_path}/right_wheel.stl" scale="${scale_mm_to_m} ${scale_mm_to_m} ${scale_mm_to_m}"/>
      </geometry>
-     <material name="black"/>
+     <material name="red"/>
    </visual>
    <collision>
@@ -117,9 +144,21 @@
        <mesh filename="${mesh_path}/right_wheel.stl" scale="${scale_mm_to_m} ${scale_mm_to_m} ${scale_mm_to_m}"/>
      </geometry>
-     <material name="black"/>
+     <material name="red"/>
+     <gazebo>
+      <material>Gazebo/Red</material>
+      <friction>
+        <ode>
+          <mu>1.0</mu>
+          <mu2>1.0</mu2>
+          <fdir1>0 1 0</fdir1>
+        </ode>
+      </friction>
+      <kp>1000000.0</kp>
+      <kd>100.0</kd>
+    </gazebo>
    </collision>
    <inertial>
-     <mass value="0.3"/>
-     <inertia ixx="0.001" ixy="0.0" ixz="0.0" iyy="0.001" iyz="0.0" izz="0.001"/>
+     <mass value="0.5"/>
+     <inertia ixx="0.00733" ixy="0.0" ixz="0.0" iyy="0.00733" iyz="0.0" izz="0.00133"/>
    </inertial>
  </link>

Commit message: rviz done

File: install/amphibious_robot_description/share/amphibious_robot_description/description/amphibot.urdf.xacro (robot description, xacro)
@@ -28,6 +28,4 @@
      <gazebo>
       <material>Gazebo/White</material>
-      <kp>1000000.0</kp>
-      <kd>100.0</kd>
     </gazebo>
    </collision>
@@ -52,6 +50,4 @@
      <gazebo>
       <material>Gazebo/Blue</material>
-      <kp>1000000.0</kp>
-      <kd>100.0</kd>
     </gazebo>
    </collision>
@@ -81,6 +77,4 @@
      <gazebo>
       <material>Gazebo/Blue</material>
-      <kp>1000000.0</kp>
-      <kd>100.0</kd>
     </gazebo>
    </collision>
@@ -110,14 +104,5 @@
      <gazebo>
       <material>Gazebo/Red</material>
-      <friction>
-        <ode>
-          <mu>1.0</mu>
-          <mu2>1.0</mu2>
-          <fdir1>0 1 0</fdir1>
-        </ode>
-      </friction>
-      <kp>1000000.0</kp>
-      <kd>100.0</kd>
-    </gazebo>
+     </gazebo>
    </collision>
    <inertial>
@@ -129,6 +114,6 @@
    <parent link="lshaft_link"/>
    <child link="left_wheel_link"/>
-   <origin xyz="0 0 .05" rpy="0 0 0" />
-   <axis xyz="0 1 0"/>
+   <origin xyz="0 0 .05" rpy="0 0 -1.5708" />
+   <axis xyz="0 0 1"/>
  </joint>
  <!-- Right Wheel -->
@@ -147,14 +132,5 @@
      <gazebo>
       <material>Gazebo/Red</material>
-      <friction>
-        <ode>
-          <mu>1.0</mu>
-          <mu2>1.0</mu2>
-          <fdir1>0 1 0</fdir1>
-        </ode>
-      </friction>
-      <kp>1000000.0</kp>
-      <kd>100.0</kd>
-    </gazebo>
+     </gazebo>
    </collision>
    <inertial>
@@ -167,5 +143,5 @@
    <child link="right_wheel_link"/>
    <origin xyz="0 0 .05" rpy="0 0 0" />
-   <axis xyz="0 1 0"/>
+   <axis xyz="0 0 1"/>
  </joint>
  </robot>

File: src/amphibious_robot_description/description/amphibot.urdf.xacro (robot description, xacro)
@@ -28,6 +28,4 @@
      <gazebo>
       <material>Gazebo/White</material>
-      <kp>1000000.0</kp>
-      <kd>100.0</kd>
     </gazebo>
    </collision>
@@ -52,6 +50,4 @@
      <gazebo>
       <material>Gazebo/Blue</material>
-      <kp>1000000.0</kp>
-      <kd>100.0</kd>
     </gazebo>
    </collision>
@@ -81,6 +77,4 @@
      <gazebo>
       <material>Gazebo/Blue</material>
-      <kp>1000000.0</kp>
-      <kd>100.0</kd>
     </gazebo>
    </collision>
@@ -110,14 +104,5 @@
      <gazebo>
       <material>Gazebo/Red</material>
-      <friction>
-        <ode>
-          <mu>1.0</mu>
-          <mu2>1.0</mu2>
-          <fdir1>0 1 0</fdir1>
-        </ode>
-      </friction>
-      <kp>1000000.0</kp>
-      <kd>100.0</kd>
-    </gazebo>
+     </gazebo>
    </collision>
    <inertial>
@@ -130,9 +115,10 @@
    <child link="left_wheel_link"/>
    <origin xyz="0 0 .05" rpy="0 0 0" />
-   <axis xyz="0 1 0"/>
+   <axis xyz="0 0 1"/>
  </joint>
  <!-- Right Wheel -->
  <link name="right_wheel_link">
    <visual>
+     <origin rpy="-1.5708 0 0"/>
      <geometry>
        <mesh filename="${mesh_path}/right_wheel.stl" scale="${scale_mm_to_m} ${scale_mm_to_m} ${scale_mm_to_m}"/>
@@ -142,4 +128,5 @@
    <collision>
      <geometry>
+       <origin rpy="-1.5708 0 0"/>
        <mesh filename="${mesh_path}/right_wheel.stl" scale="${scale_mm_to_m} ${scale_mm_to_m} ${scale_mm_to_m}"/>
      </geometry>
@@ -147,14 +134,5 @@
      <gazebo>
       <material>Gazebo/Red</material>
-      <friction>
-        <ode>
-          <mu>1.0</mu>
-          <mu2>1.0</mu2>
-          <fdir1>0 1 0</fdir1>
-        </ode>
-      </friction>
-      <kp>1000000.0</kp>
-      <kd>100.0</kd>
-    </gazebo>
+     </gazebo>
    </collision>
    <inertial>
@@ -167,5 +145,5 @@
    <child link="right_wheel_link"/>
    <origin xyz="0 0 .05" rpy="0 0 0" />
-   <axis xyz="0 1 0"/>
+   <axis xyz="0 0 1"/>
  </joint>
  </robot>

Commit message: rviz

File: install/amphibious_robot_description/share/amphibious_robot_description/description/amphibot.urdf.xacro (robot description, xacro)
@@ -45,5 +45,5 @@
    <collision>
      <geometry>
-       <mesh filename="${mesh_path}/shaft.stl" scale="${scale_mm_to_m} ${scale_mm_to_m} ${scale_mm_to_m}"/>
+       <mesh filename="${mesh_path}/rshaft.stl" scale="${scale_mm_to_m} ${scale_mm_to_m} ${scale_mm_to_m}"/>
      </geometry>
      <material name="blue"/>
@@ -66,5 +66,5 @@
    <visual>
      <geometry>
-       <mesh filename="${mesh_path}/shaft.stl" scale="${scale_mm_to_m} ${scale_mm_to_m} ${scale_mm_to_m}"/>
+       <mesh filename="${mesh_path}/lshaft.stl" scale="${scale_mm_to_m} ${scale_mm_to_m} ${scale_mm_to_m}"/>
      </geometry>
      <material name="blue"/>
@@ -114,5 +114,5 @@
    <parent link="lshaft_link"/>
    <child link="left_wheel_link"/>
-   <origin xyz="0 0 .05" rpy="0 0 -1.5708" />
+   <origin xyz="0 0 .05" rpy="0 0 0" />
    <axis xyz="0 0 1"/>
  </joint>

File: src/amphibious_robot_description/description/amphibot.urdf.xacro (robot description, xacro)
@@ -45,5 +45,5 @@
    <collision>
      <geometry>
-       <mesh filename="${mesh_path}/shaft.stl" scale="${scale_mm_to_m} ${scale_mm_to_m} ${scale_mm_to_m}"/>
+       <mesh filename="${mesh_path}/rshaft.stl" scale="${scale_mm_to_m} ${scale_mm_to_m} ${scale_mm_to_m}"/>
      </geometry>
      <material name="blue"/>
@@ -66,5 +66,5 @@
    <visual>
      <geometry>
-       <mesh filename="${mesh_path}/shaft.stl" scale="${scale_mm_to_m} ${scale_mm_to_m} ${scale_mm_to_m}"/>
+       <mesh filename="${mesh_path}/lshaft.stl" scale="${scale_mm_to_m} ${scale_mm_to_m} ${scale_mm_to_m}"/>
      </geometry>
      <material name="blue"/>
@@ -120,5 +120,4 @@
  <link name="right_wheel_link">
    <visual>
-     <origin rpy="-1.5708 0 0"/>
      <geometry>
        <mesh filename="${mesh_path}/right_wheel.stl" scale="${scale_mm_to_m} ${scale_mm_to_m} ${scale_mm_to_m}"/>
@@ -128,5 +127,4 @@
    <collision>
      <geometry>
-       <origin rpy="-1.5708 0 0"/>
        <mesh filename="${mesh_path}/right_wheel.stl" scale="${scale_mm_to_m} ${scale_mm_to_m} ${scale_mm_to_m}"/>
      </geometry>

Commit message: spawned bot in world

File: install/amphibious_robot_description/share/amphibious_robot_description/description/amphibot.urdf.xacro (robot description, xacro)
@@ -11,5 +11,5 @@
    </material>
  <!-- Robot-wide properties -->
- <xacro:property name="mesh_path" value="package://amphibious_robot_description/meshes"/>
+ <xacro:property name="mesh_path" value="model://amphibious_robot_description/meshes"/>
  <xacro:property name="scale_mm_to_m" value="0.001"/>
  <!-- Body -->

Commit message: spawned bot in the world

File: install/amphibious_robot_description/share/amphibious_robot_description/description/amphibot.urdf.xacro (robot description, xacro)
@@ -11,5 +11,5 @@
    </material>
  <!-- Robot-wide properties -->
- <xacro:property name="mesh_path" value="model://amphibious_robot_description/meshes"/>
+ <xacro:property name="mesh_path" value="package://amphibious_robot_description/meshes"/>
  <xacro:property name="scale_mm_to_m" value="0.001"/>
  <!-- Body -->
